File: kicad/SolatronG2U.kicad_pcb (KiCad board)
At the start: 2 copper layers, 34 parts, among them J1 Conn_02x12_Counter_Clockwise_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

Commit message: Added new footprint for Centronics
Parts:
- added REF**: MountingHole_3.2mm_M3, MountingHole:MountingHole_3.2mm_M3, F.Cu at (132.7, 31.1)
- added REF**: MountingHole_3.2mm_M3, MountingHole:MountingHole_3.2mm_M3, F.Cu at (197.2, 31.1)
- added REF**: MountingHole_3.2mm_M3, MountingHole:MountingHole_3.2mm_M3, F.Cu at (132.7, 101.0)
- added REF**: MountingHole_3.2mm_M3, MountingHole:MountingHole_3.2mm_M3, F.Cu at (197.2, 101.0)
Routing:
- net Net-(A1-A0): track 64.1 -> 59.9 mm
- net Net-(A1-A2): track 93.2 -> 89.9 mm
- net Net-(A1-A3): track 109.1 -> 106.0 mm
- net GND: track 134.0 -> 132.3 mm
- added copper zone on B.Cu, net GND
Other:
- board outline added: 73.6 x 78.7 mm
